Commit message: fine-tune URDF

File: witdog_description/urdf/witdog_description.urdf (robot description, URDF)
Before this commit: robot witdog, 19 links, 18 joints
Joints:
- joint to_lf3: origin xyz=-0.00091985 0.0079405 -0.066613 rpy=0 0 0 -> xyz=-0.00091985 0.0079405 -0.060 rpy=0 0 0
- joint to_lh3: origin xyz=-0.000919847336912388 0.00794054054057377 -0.0666130631353466 rpy=0 0 0 -> xyz=-0.000919847336912388 0.00794054054057377 -0.060 rpy=0 0 0
- joint to_rf3: origin xyz=-0.000919872443398681 -0.00834054054053998 -0.0666128977412097 rpy=0 0 0 -> xyz=-0.000919872443398681 -0.00834054054053998 -0.060 rpy=0 0 0
- joint to_rh3: origin xyz=-0.000919872443398723 -0.00834054054054026 -0.0666128977412097 rpy=0 0 0 -> xyz=-0.000919872443398723 -0.00834054054054026 -0.060 rpy=0 0 0
